File: digital_lockin_LOOK_AT_THIS.brd (EAGLE design)
At the start: 76.2 x 94.9 mm, 24 parts, among them IC1 OPA2650E, IC2 LM358D, T2 NPN, U2 RASPBERRY_PICOSMD-TH, U5 TL431AIDBZR

Commit message: UPLOAD
look at this when i upload
Parts:
- moved R9 39.3 mm to (26.2, 3.56)
- moved R7 19.8 mm to (56.1, 3.56)
- moved R3 16.8 mm to (35.8, 21.3)
- moved C1 16.7 mm to (41.9, 20.8)
- moved C10 15.9 mm to (40.1, 15.2)
- moved C8 14.7 mm to (59.4, 19.3)
- moved PD1 14.3 mm to (31.8, 10.4)
- moved C2 12.4 mm to (53.1, 10.4)
- moved C3 10.6 mm to (69.3, 12.2)
- moved IC1 8.68 mm to (50.8, 16.0)
- moved R6 6.43 mm to (59.7, 27.9)
- moved R5 6.12 mm to (50.5, 25.7)
- moved C9 1.83 mm to (22.4, 48.8)
Routing:
- net 5V: track 0.00 -> 185.8 mm
- net ADCMID: track 0.00 -> 153.6 mm
- net GND: track 0.00 -> 72.1 mm, vias 4 -> 6
- net AMPOUT: track 0.00 -> 71.4 mm
- net LEDCTRL: track 0.00 -> 67.4 mm, vias 0 -> 2
- net 3V3: track 0.00 -> 60.0 mm
- net ADCREF: track 0.00 -> 55.8 mm
- net N$5: track 0.00 -> 46.3 mm
- net N$1: track 0.00 -> 43.9 mm
- net N$7: track 0.00 -> 27.9 mm
- net N$9: track 0.00 -> 16.4 mm
- net N$2: track 0.00 -> 14.6 mm
- net N$10: track 0.00 -> 11.1 mm
- net N$20: track 0.00 -> 7.35 mm
- net N$3: track 0.00 -> 5.65 mm
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- added copper zone on layer 16, net GND
